Commit message: adjust the urdf output path, also for testing github

File: examples/snake/bb_snake.urdf (robot description, URDF)
Before this commit: robot bb_snake, 83 links, 82 joints
Links:
- removed link act0Seg10
- removed link act0Seg10helper_shape
- removed link act0Seg11
- removed link act0Seg11helper_shape
- removed link act0Seg12
- removed link act0Seg12helper_shape
- removed link act0Seg13
- removed link act0Seg13helper_shape
- removed link act0Seg14
- removed link act0Seg14helper_shape
- removed link act0Seg15
- removed link act0Seg15helper_shape
- removed link act0Seg16
- removed link act0Seg16helper_shape
- removed link act0Seg17
- removed link act0Seg17helper_shape
- removed link act0Seg18
- removed link act0Seg18helper_shape
- removed link act0Seg19
- removed link act0Seg19helper_shape
- removed link act0Seg20
- removed link act0Seg20helper_shape
- removed link act0Seg9
- removed link act0Seg9helper_shape
- removed link act1Seg10
- removed link act1Seg10helper_shape
- removed link act1Seg11
- removed link act1Seg11helper_shape
- removed link act1Seg12
- removed link act1Seg12helper_shape
- removed link act1Seg13
- removed link act1Seg13helper_shape
- removed link act1Seg14
- removed link act1Seg14helper_shape
- removed link act1Seg15
- removed link act1Seg15helper_shape
- removed link act1Seg16
- removed link act1Seg16helper_shape
- removed link act1Seg17
- removed link act1Seg17helper_shape
- removed link act1Seg18
- removed link act1Seg18helper_shape
- removed link act1Seg19
- removed link act1Seg19helper_shape
- removed link act1Seg20
- removed link act1Seg20helper_shape
- removed link act1Seg9
- removed link act1Seg9helper_shape
- link act0Seg0: geometry collision box size=0.12 0.12 0.05; visual box size=0.12 0.12 0.05
- link act0Seg1: geometry collision box size=0.12 0.12 0.1; visual box size=0.12 0.12 0.1
- link act0Seg1helper_shape: geometry collision cylinder length=0.12 radius=0.06; visual cylinder length=0.12 radius=0.06
- link act0Seg2: geometry collision box size=0.12 0.12 0.1; visual box size=0.12 0.12 0.1
- link act0Seg2helper_shape: geometry collision cylinder length=0.12 radius=0.06; visual cylinder length=0.12 radius=0.06
- link act0Seg3: geometry collision box size=0.12 0.12 0.1; visual box size=0.12 0.12 0.1
- link act0Seg3helper_shape: geometry collision cylinder length=0.12 radius=0.06; visual cylinder length=0.12 radius=0.06
- link act0Seg4: geometry collision box size=0.12 0.12 0.1; visual box size=0.12 0.12 0.1
- link act0Seg4helper_shape: geometry collision cylinder length=0.12 radius=0.06; visual cylinder length=0.12 radius=0.06
- link act0Seg5: geometry collision box size=0.12 0.12 0.1; visual box size=0.12 0.12 0.1
- link act0Seg5helper_shape: geometry collision cylinder length=0.12 radius=0.06; visual cylinder length=0.12 radius=0.06
- link act0Seg6: geometry collision box size=0.12 0.12 0.1; visual box size=0.12 0.12 0.1
- link act0Seg6helper_shape: geometry collision cylinder length=0.12 radius=0.06; visual cylinder length=0.12 radius=0.06
- link act0Seg7: geometry collision box size=0.12 0.12 0.1; visual box size=0.12 0.12 0.1
- link act0Seg7helper_shape: geometry collision cylinder length=0.12 radius=0.06; visual cylinder length=0.12 radius=0.06
- link act0Seg8: geometry collision box size=0.12 0.12 0.05; visual box size=0.12 0.12 0.05
- link act0Seg8helper_shape: geometry collision cylinder length=0.12 radius=0.06; visual cylinder length=0.12 radius=0.06
- link act1Seg0: geometry collision box size=0.12 0.12 0.05; visual box size=0.12 0.12 0.05
- link act1Seg1: geometry collision box size=0.12 0.12 0.1; visual box size=0.12 0.12 0.1
- link act1Seg1helper_shape: geometry collision cylinder length=0.12 radius=0.06; visual cylinder length=0.12 radius=0.06
- link act1Seg2: geometry collision box size=0.12 0.12 0.1; visual box size=0.12 0.12 0.1
- link act1Seg2helper_shape: geometry collision cylinder length=0.12 radius=0.06; visual cylinder length=0.12 radius=0.06
- link act1Seg3: geometry collision box size=0.12 0.12 0.1; visual box size=0.12 0.12 0.1
- link act1Seg3helper_shape: geometry collision cylinder length=0.12 radius=0.06; visual cylinder length=0.12 radius=0.06
- link act1Seg4: geometry collision box size=0.12 0.12 0.1; visual box size=0.12 0.12 0.1
- link act1Seg4helper_shape: geometry collision cylinder length=0.12 radius=0.06; visual cylinder length=0.12 radius=0.06
- link act1Seg5: geometry collision box size=0.12 0.12 0.1; visual box size=0.12 0.12 0.1
- link act1Seg5helper_shape: geometry collision cylinder length=0.12 radius=0.06; visual cylinder length=0.12 radius=0.06
- link act1Seg6: geometry collision box size=0.12 0.12 0.1; visual box size=0.12 0.12 0.1
- link act1Seg6helper_shape: geometry collision cylinder length=0.12 radius=0.06; visual cylinder length=0.12 radius=0.06
- link act1Seg7: geometry collision box size=0.12 0.12 0.1; visual box size=0.12 0.12 0.1
- link act1Seg7helper_shape: geometry collision cylinder length=0.12 radius=0.06; visual cylinder length=0.12 radius=0.06
- link act1Seg8: geometry collision box size=0.12 0.12 0.05; visual box size=0.12 0.12 0.05
- link act1Seg8helper_shape: geometry collision cylinder length=0.12 radius=0.06; visual cylinder length=0.12 radius=0.06
Joints:
- removed joint act0Seg10_to_act0Seg11_ax0
- removed joint act0Seg10_to_act0Seg11_ax0helper_shape
- removed joint act0Seg11_to_act0Seg12_ax1
- removed joint act0Seg11_to_act0Seg12_ax1helper_shape
- removed joint act0Seg12_to_act0Seg13_ax0
- removed joint act0Seg12_to_act0Seg13_ax0helper_shape
- removed joint act0Seg13_to_act0Seg14_ax1
- removed joint act0Seg13_to_act0Seg14_ax1helper_shape
- removed joint act0Seg14_to_act0Seg15_ax0
- removed joint act0Seg14_to_act0Seg15_ax0helper_shape
- removed joint act0Seg15_to_act0Seg16_ax1
- removed joint act0Seg15_to_act0Seg16_ax1helper_shape
- removed joint act0Seg16_to_act0Seg17_ax0
- removed joint act0Seg16_to_act0Seg17_ax0helper_shape
- removed joint act0Seg17_to_act0Seg18_ax1
- removed joint act0Seg17_to_act0Seg18_ax1helper_shape
- removed joint act0Seg18_to_act0Seg19_ax0
- removed joint act0Seg18_to_act0Seg19_ax0helper_shape
- removed joint act0Seg19_to_act0Seg20_ax1
- removed joint act0Seg19_to_act0Seg20_ax1helper_shape
- removed joint act0Seg20_to_act1Seg0_ax1
- removed joint act0Seg8_to_act0Seg9_ax0
- removed joint act0Seg8_to_act0Seg9_ax0helper_shape
- removed joint act0Seg9_to_act0Seg10_ax1
- removed joint act0Seg9_to_act0Seg10_ax1helper_shape
- removed joint act1Seg10_to_act1Seg11_ax0
- removed joint act1Seg10_to_act1Seg11_ax0helper_shape
- removed joint act1Seg11_to_act1Seg12_ax1
- removed joint act1Seg11_to_act1Seg12_ax1helper_shape
- removed joint act1Seg12_to_act1Seg13_ax0
- removed joint act1Seg12_to_act1Seg13_ax0helper_shape
- removed joint act1Seg13_to_act1Seg14_ax1
- removed joint act1Seg13_to_act1Seg14_ax1helper_shape
- removed joint act1Seg14_to_act1Seg15_ax0
- removed joint act1Seg14_to_act1Seg15_ax0helper_shape
- removed joint act1Seg15_to_act1Seg16_ax1
- removed joint act1Seg15_to_act1Seg16_ax1helper_shape
- removed joint act1Seg16_to_act1Seg17_ax0
- removed joint act1Seg16_to_act1Seg17_ax0helper_shape
- removed joint act1Seg17_to_act1Seg18_ax1
- removed joint act1Seg17_to_act1Seg18_ax1helper_shape
- removed joint act1Seg18_to_act1Seg19_ax0
- removed joint act1Seg18_to_act1Seg19_ax0helper_shape
- removed joint act1Seg19_to_act1Seg20_ax1
- removed joint act1Seg19_to_act1Seg20_ax1helper_shape
- removed joint act1Seg8_to_act1Seg9_ax0
- removed joint act1Seg8_to_act1Seg9_ax0helper_shape
- removed joint act1Seg9_to_act1Seg10_ax1
- removed joint act1Seg9_to_act1Seg10_ax1helper_shape
- added joint act0Seg8_to_act1Seg0_ax1: type fixed, parent act0Seg8, child act1Seg0, origin xyz=0 0 0.05 rpy=0 0 0, axis 0 1 0, limit lower=-0.785398 upper=0.785398 effort=100 velocity=3
- joint act0Seg0_to_act0Seg1_ax0: origin xyz=0 0 0.0245 rpy=0 0 0 -> xyz=0 0 0.05 rpy=0 0 0
- joint act0Seg0_to_act0Seg1_ax0helper_shape: origin xyz=0 0 0.0245 rpy=0 0 0 -> xyz=0 0 0.05 rpy=0 0 0
- joint act0Seg1_to_act0Seg2_ax1: origin xyz=0 0 0.049 rpy=0 0 0 -> xyz=0 0 0.1 rpy=0 0 0
- joint act0Seg1_to_act0Seg2_ax1helper_shape: origin xyz=0 0 0.049 rpy=0 0 0 -> xyz=0 0 0.1 rpy=0 0 0
- joint act0Seg2_to_act0Seg3_ax0: origin xyz=0 0 0.049 rpy=0 0 0 -> xyz=0 0 0.1 rpy=0 0 0
- joint act0Seg2_to_act0Seg3_ax0helper_shape: origin xyz=0 0 0.049 rpy=0 0 0 -> xyz=0 0 0.1 rpy=0 0 0
- joint act0Seg3_to_act0Seg4_ax1: origin xyz=0 0 0.049 rpy=0 0 0 -> xyz=0 0 0.1 rpy=0 0 0
- joint act0Seg3_to_act0Seg4_ax1helper_shape: origin xyz=0 0 0.049 rpy=0 0 0 -> xyz=0 0 0.1 rpy=0 0 0
- joint act0Seg4_to_act0Seg5_ax0: origin xyz=0 0 0.049 rpy=0 0 0 -> xyz=0 0 0.1 rpy=0 0 0
- joint act0Seg4_to_act0Seg5_ax0helper_shape: origin xyz=0 0 0.049 rpy=0 0 0 -> xyz=0 0 0.1 rpy=0 0 0
- joint act0Seg5_to_act0Seg6_ax1: origin xyz=0 0 0.049 rpy=0 0 0 -> xyz=0 0 0.1 rpy=0 0 0
- joint act0Seg5_to_act0Seg6_ax1helper_shape: origin xyz=0 0 0.049 rpy=0 0 0 -> xyz=0 0 0.1 rpy=0 0 0
- joint act0Seg6_to_act0Seg7_ax0: origin xyz=0 0 0.049 rpy=0 0 0 -> xyz=0 0 0.1 rpy=0 0 0
- joint act0Seg6_to_act0Seg7_ax0helper_shape: origin xyz=0 0 0.049 rpy=0 0 0 -> xyz=0 0 0.1 rpy=0 0 0
- joint act0Seg7_to_act0Seg8_ax1: origin xyz=0 0 0.049 rpy=0 0 0 -> xyz=0 0 0.1 rpy=0 0 0
- joint act0Seg7_to_act0Seg8_ax1helper_shape: origin xyz=0 0 0.049 rpy=0 0 0 -> xyz=0 0 0.1 rpy=0 0 0
- joint act1Seg0_to_act1Seg1_ax0: origin xyz=0 0 0.0245 rpy=0 0 0 -> xyz=0 0 0.05 rpy=0 0 0
- joint act1Seg0_to_act1Seg1_ax0helper_shape: origin xyz=0 0 0.0245 rpy=0 0 0 -> xyz=0 0 0.05 rpy=0 0 0
- joint act1Seg1_to_act1Seg2_ax1: origin xyz=0 0 0.049 rpy=0 0 0 -> xyz=0 0 0.1 rpy=0 0 0
- joint act1Seg1_to_act1Seg2_ax1helper_shape: origin xyz=0 0 0.049 rpy=0 0 0 -> xyz=0 0 0.1 rpy=0 0 0
- joint act1Seg2_to_act1Seg3_ax0: origin xyz=0 0 0.049 rpy=0 0 0 -> xyz=0 0 0.1 rpy=0 0 0
- joint act1Seg2_to_act1Seg3_ax0helper_shape: origin xyz=0 0 0.049 rpy=0 0 0 -> xyz=0 0 0.1 rpy=0 0 0
- joint act1Seg3_to_act1Seg4_ax1: origin xyz=0 0 0.049 rpy=0 0 0 -> xyz=0 0 0.1 rpy=0 0 0
- joint act1Seg3_to_act1Seg4_ax1helper_shape: origin xyz=0 0 0.049 rpy=0 0 0 -> xyz=0 0 0.1 rpy=0 0 0
- joint act1Seg4_to_act1Seg5_ax0: origin xyz=0 0 0.049 rpy=0 0 0 -> xyz=0 0 0.1 rpy=0 0 0
- joint act1Seg4_to_act1Seg5_ax0helper_shape: origin xyz=0 0 0.049 rpy=0 0 0 -> xyz=0 0 0.1 rpy=0 0 0
- joint act1Seg5_to_act1Seg6_ax1: origin xyz=0 0 0.049 rpy=0 0 0 -> xyz=0 0 0.1 rpy=0 0 0
- joint act1Seg5_to_act1Seg6_ax1helper_shape: origin xyz=0 0 0.049 rpy=0 0 0 -> xyz=0 0 0.1 rpy=0 0 0
- joint act1Seg6_to_act1Seg7_ax0: origin xyz=0 0 0.049 rpy=0 0 0 -> xyz=0 0 0.1 rpy=0 0 0
- joint act1Seg6_to_act1Seg7_ax0helper_shape: origin xyz=0 0 0.049 rpy=0 0 0 -> xyz=0 0 0.1 rpy=0 0 0
- joint act1Seg7_to_act1Seg8_ax1: origin xyz=0 0 0.049 rpy=0 0 0 -> xyz=0 0 0.1 rpy=0 0 0
- joint act1Seg7_to_act1Seg8_ax1helper_shape: origin xyz=0 0 0.049 rpy=0 0 0 -> xyz=0 0 0.1 rpy=0 0 0
