Commit message: small changes

File: examples/snake/bb_snake1.urdf (robot description, URDF)
Before this commit: robot bb_snake, 21 links, 20 joints
Joints:
- added joint act0Seg0_to_act1Seg0: type fixed, parent act0Seg0, child act1Seg0, origin xyz=0 0 0.05 rpy=0 0 0, axis 1 0 0, limit lower=0 upper=0 effort=100 velocity=3
- added joint act1Seg0_to_act2Seg0: type fixed, parent act1Seg0, child act2Seg0, origin xyz=0 0 0.05 rpy=0 0 0, axis 1 0 0, limit lower=0 upper=0 effort=100 velocity=3
- added joint act2Seg0_to_act3Seg0: type fixed, parent act2Seg0, child act3Seg0, origin xyz=0 0 0.05 rpy=0 0 0, axis 1 0 0, limit lower=0 upper=0 effort=100 velocity=3
- joint act0Seg0_to_act0Seg1_ax0: type revolute -> fixed

Commit message: iteration implemented

File: examples/snake/bb_snake1.urdf (robot description, URDF)
Before this commit: robot bb_snake, 21 links, 23 joints
Links:
- removed link act2Seg0
- removed link act2Seg1
- removed link act2Seg1helper_shape
- removed link act2Seg2
- removed link act2Seg2helper_shape
- removed link act3Seg0
- removed link act3Seg1
- removed link act3Seg1helper_shape
- removed link act3Seg2
- removed link act3Seg2helper_shape
Joints:
- removed joint act0Seg0_to_act1Seg0
- removed joint act0Seg1_to_act1Seg1_ax1
- removed joint act1Seg0_to_act2Seg0
- removed joint act1Seg1_to_act2Seg1_ax1
- removed joint act2Seg0_to_act2Seg1_ax0
- removed joint act2Seg0_to_act2Seg1_ax0helper_shape
- removed joint act2Seg0_to_act3Seg0
- removed joint act2Seg1_to_act2Seg2_ax1
- removed joint act2Seg1_to_act2Seg2_ax1helper_shape
- removed joint act2Seg1_to_act3Seg1_ax1
- removed joint act3Seg0_to_act3Seg1_ax0
- removed joint act3Seg0_to_act3Seg1_ax0helper_shape
- removed joint act3Seg1_to_act3Seg2_ax1
- removed joint act3Seg1_to_act3Seg2_ax1helper_shape
- added joint act1Seg0_to_act0Seg0: type fixed, parent act0Seg0, child act1Seg0, origin xyz=0 0 0 rpy=0 0 0, axis 0 1 0
- joint act0Seg0_to_act0Seg1_ax0: type fixed -> revolute
